File: FitLensPCB.kicad_pcb (KiCad board)
At the start: 2 copper layers, 75 parts, among them J1 nRF debug, J10 1x1, J11 Conn_Coaxial, J12 Conn_01x02_Pin, J13 Conn_01x04_Socket, J14 Conn_Coaxial, J15 nRF debug, J5 Conn_Pin, J6 Conn_01x03_Pin, J7 1x1, J8 1x1, J9 1x1, Q2 AO3401A, SW1 SW_MEC_5G, U1 MCP73831-2-OT, U10 MAX17048G_T10, U4 STM32WB55RGVx, U6 AT42QT1010-TSHR, U7 AT42QT1010-TSHR, U8 74AHC1G08, U9 5186, Y1 32mHz, Y2 32.768kHz

Commit message: screw this
Parts:
- removed J14: Conn_Coaxial, Connector_Coaxial:U.FL_Hirose_U.FL-R-SMT-1_Vertical
- added C20: 100nF, Capacitor_SMD:C_1206_3216Metric_Pad1.33x1.80mm_HandSolder, B.Cu at (112.0, 65.5)
- added C21: 100nF, Capacitor_SMD:C_1206_3216Metric_Pad1.33x1.80mm_HandSolder, B.Cu at (178.5, 93.0)
- added C22: 100nF, Capacitor_SMD:C_1206_3216Metric_Pad1.33x1.80mm_HandSolder, B.Cu at (182.5, 89.0)
- added C23: 1uF, Capacitor_SMD:C_1206_3216Metric_Pad1.33x1.80mm_HandSolder, B.Cu at (176.5, 95.0)
- added C24: 10uF, Capacitor_SMD:C_1206_3216Metric_Pad1.33x1.80mm_HandSolder, B.Cu at (202.5, 69.5)
- added C32: 100nF, Capacitor_SMD:C_1206_3216Metric_Pad1.33x1.80mm_HandSolder, F.Cu at (147.6, 73.0)
- added C34: 4.7uF, Capacitor_SMD:C_1206_3216Metric_Pad1.33x1.80mm_HandSolder, B.Cu at (187.0, 93.5)
- added J2: Conn_01x02_Pin, Connector_JST:JST_PH_B2B-PH-K_1x02_P2.00mm_Vertical, F.Cu at (107.5, 79.5)
- added J3: USB_C_Receptacle_USB2.0_16P, Connector_USB:USB_C_Receptacle_Amphenol_12401548E4-2A, F.Cu at (108.5, 87.5)
- added R10: 56k, Resistor_SMD:R_0805_2012Metric_Pad1.20x1.40mm_HandSolder, F.Cu at (204.0, 79.0)
- added R11: 10k, Resistor_SMD:R_0805_2012Metric_Pad1.20x1.40mm_HandSolder, F.Cu at (213.0, 81.9)
- added R13: 10k, Resistor_SMD:R_0805_2012Metric_Pad1.20x1.40mm_HandSolder, F.Cu at (213.0, 84.8)
- added R14: 1k, Resistor_SMD:R_0805_2012Metric_Pad1.20x1.40mm_HandSolder, B.Cu at (116.5, 60.0)
- added R15: 10k, Resistor_SMD:R_0805_2012Metric_Pad1.20x1.40mm_HandSolder, F.Cu at (213.0, 90.8)
- added R16: 10k, Resistor_SMD:R_0805_2012Metric_Pad1.20x1.40mm_HandSolder, F.Cu at (213.0, 93.7)
- added R22: 1M, Capacitor_SMD:C_0805_2012Metric_Pad1.18x1.45mm_HandSolder, F.Cu at (117.5, 90.5)
- added R26: 10k, Resistor_SMD:R_0805_2012Metric_Pad1.20x1.40mm_HandSolder, F.Cu at (213.0, 96.7)
- added R28: 10k, Resistor_SMD:R_0805_2012Metric_Pad1.20x1.40mm_HandSolder, B.Cu at (176.5, 83.0)
- added R8: 10k, Resistor_SMD:R_0805_2012Metric_Pad1.20x1.40mm_HandSolder, F.Cu at (193.0, 58.5)
- added U11: TPD2EUSB30, Package_TO_SOT_SMD:Texas_DRT-3, F.Cu at (115.6, 87.5)
- added U12: MAX6816, Package_TO_SOT_SMD:SOT-143, F.Cu at (181.5, 69.5)
- C10, C3, C4, C5, C6, C7, C8, C9: footprint Capacitor_SMD:C_0805_2012Metric -> Capacitor_SMD:C_1206_3216Metric_Pad1.33x1.80mm_HandSolder
- C12, C13, C30: footprint Capacitor_SMD:C_0603_1608Metric_Pad1.08x0.95mm_HandSolder -> Capacitor_SMD:C_1206_3216Metric_Pad1.33x1.80mm_HandSolder; moved to B.Cu
- C14, C15, C16, C17, C26, C27, C28, C29: footprint Capacitor_SMD:C_0603_1608Metric_Pad1.08x0.95mm_HandSolder -> Capacitor_SMD:C_1206_3216Metric_Pad1.33x1.80mm_HandSolder
- C18, C19: footprint Capacitor_SMD:C_01005_0402Metric_Pad0.57x0.30mm_HandSolder -> Capacitor_SMD:C_1206_3216Metric_Pad1.33x1.80mm_HandSolder
- C31: value 100nF -> 2.2uF; footprint Capacitor_SMD:C_0603_1608Metric_Pad1.08x0.95mm_HandSolder -> Capacitor_SMD:C_1206_3216Metric_Pad1.33x1.80mm_HandSolder; moved to B.Cu
- D2, D3: moved to B.Cu
- D5: value 1N4148W -> LED; footprint Diode_SMD:D_SOD-123 -> LED_SMD:LED_0805_2012Metric
- D7: value SB120 -> SS12; footprint Diode_THT:D_DO-41_SOD81_P10.16mm_Horizontal -> Diode_SMD:D_SOD-123F
- D8: value SB120 -> SS12; footprint Diode_THT:D_DO-41_SOD81_P10.16mm_Horizontal -> Diode_SMD:D_SOD-123F; moved to B.Cu
- J11: value Conn_Coaxial -> Conn_01x05_Pin; footprint Connector_Coaxial:U.FL_Hirose_U.FL-R-SMT-1_Vertical -> Connector_Hirose:Hirose_DF13-05P-1.25DS_1x05_P1.25mm_Horizontal
- R1, R2, R3, R4, R7: footprint Resistor_SMD:R_0603_1608Metric -> Resistor_SMD:R_0805_2012Metric_Pad1.20x1.40mm_HandSolder
- R12, R9: footprint Resistor_SMD:R_0603_1608Metric_Pad0.98x0.95mm_HandSolder -> Resistor_SMD:R_0805_2012Metric_Pad1.20x1.40mm_HandSolder
- R18, R19, R20: footprint Resistor_SMD:R_0201_0603Metric_Pad0.64x0.40mm_HandSolder -> Resistor_SMD:R_0805_2012Metric_Pad1.20x1.40mm_HandSolder
- R5, R6: footprint Resistor_SMD:R_0603_1608Metric -> Resistor_SMD:R_0805_2012Metric_Pad1.20x1.40mm_HandSolder; moved to B.Cu
- SW1: footprint Button_Switch_SMD:SW_MEC_5GSH9 -> Button_Switch_SMD:SW_Push_1P1T_NO_CK_KSC7xxJ
- U9: value 5186 -> CD-PA1616D; footprint PA1616D:CD-PA1616D_ADA -> CD-PA1616D:XCVR_CD-PA1616D
- moved J12 118.9 mm to (232.5, 65.0), turned to 90 degrees
- moved J5 98.2 mm to (232.8, 87.5), turned to 90 degrees
- moved J13 91.7 mm to (228.0, 123.5)
- moved E1 88.3 mm to (202.6, 63.8)
- moved J6 85.0 mm to (233.0, 76.0), turned to 90 degrees
- moved J1 82.8 mm to (230.4, 95.0)
- moved J15 82.7 mm to (230.4, 104.0)
- moved J11 62.8 mm to (210.0, 111.5)
- moved D7 58.9 mm to (191.5, 62.5)
- moved SW1 53.6 mm to (180.1, 61.5)
- moved D5 53.3 mm to (127.5, 58.5), turned to -90 degrees
- moved D3 51.5 mm to (116.0, 83.5), turned to -90 degrees
- moved L1 49.3 mm to (153.0, 151.0)
- moved C3 48.0 mm to (157.5, 120.5)
- moved C5 48.0 mm to (157.5, 126.5)
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Connections:
- net /GPS_NRST renamed /nRST_GPS
- D5 pad 1: /UART1_TX -> -BATT
- J11 pad 1: Net-(J11-In) -> +VCC_OUT
- J11 pad 2: -BATT -> /BOOT0
- U10 pad 7: /I2C1_SCL -> /I2C_SCL
- U4 pad 1: unconnected-(U4-VBAT-Pad1) -> +VCC_OUT
- U4 pad 10: /QSPI_IO3 -> /GPS_RX
- U4 pad 19: unconnected-(U4-PA4-Pad19) -> /BAT_ALERT
- U4 pad 5: unconnected-(U4-PH3-Pad5) -> /BOOT0
- U4 pad 8: unconnected-(U4-NRST-Pad8) -> /nRST_STM
- U4 pad 9: /QSPI_IO2 -> /GPS_TX
- U9 pad 1: +VCC_OUT -> Net-(Q4-S)
- U9 pad 10: Net-(U9-RX0) -> /GPS_RX
- U9 pad 11: Net-(J11-In) -> unconnected-(U9-EX_ANT-Pad11)
- U9 pad 13: unconnected-(U9-1PPS-Pad13) -> /GPS_1PPS
- U9 pad 5: Net-(D6-A) -> /GPS_FIX
- U9 pad 9: Net-(U9-TX0) -> /GPS_TX
Routing:
- net -BATT: track 0.00 -> 101.3 mm, vias 0 -> 14
- net +VCC_OUT: track 0.00 -> 33.5 mm, vias 0 -> 10
- net Net-(D7-K): track 0.00 -> 29.1 mm, vias 0 -> 1
- net Net-(J3-SHIELD): track 0.00 -> 28.6 mm
- net /nRST_nRF: track 0.00 -> 17.5 mm
- net +BATT: track 0.00 -> 15.5 mm
- net Net-(J3-CC1): track 0.00 -> 14.9 mm, vias 0 -> 1
- net /nRST_STM: track 0.00 -> 14.8 mm, vias 0 -> 1
- net /GPS_FIX: track 0.00 -> 10.9 mm, vias 0 -> 1
- net Net-(D5-A): track 0.00 -> 10.3 mm, vias 0 -> 1
- net Net-(D2-A2): track 0.00 -> 8.18 mm, vias 0 -> 1
- net /USB_DM: track 0.00 -> 7.57 mm, vias 0 -> 1
- net Net-(J3-CC2): track 0.00 -> 4.44 mm
- net VBUS: track 0.00 -> 4.31 mm, vias 0 -> 1
- net /USB_DP: track 0.00 -> 3.25 mm
- added copper zone on B.Cu, net +VCC_OUT
- added copper zone on In2.Cu, net +VCC_OUT
- added copper zone on In1.Cu, net -BATT
Other:
- board outline added: 130 x 59.5 mm
- copper layers 2 -> 4
- board text added: "LDR"
- board text added: "Touch Sensors"

Commit message: lol
Parts:
- removed D6: LED, LED_SMD:LED_0603_1608Metric_Pad1.05x0.95mm_HandSolder
- added Q1: FS8205A, FS8205A:SOP65P640X120-8N, F.Cu at (123.6, 76.5)
- added Q3: PMOS, Package_TO_SOT_SMD:SOT-723, F.Cu at (171.1, 97.0)
- added Q4: PMOS, Package_TO_SOT_SMD:SOT-723, B.Cu at (110.0, 58.5)
- added U2: DW01A, DW01A:SOT95P280X145-6N, F.Cu at (116.0, 76.5)
- added U3: TPS63020DSJR, TPS63020DSJR:IC_TPS63020DSJR, F.Cu at (136.5, 83.5)
- added U5: MX25L3233FM1, MX25L3233FM2I-08G:SOIC127P790X216-8N_MX25L3233FM2I-08G, F.Cu at (164.0, 99.0)
- C10, C14, C28, C3, C7, C8, C9, R1, R13, R16, R3, R4: moved to B.Cu
- C21, C23, C30, C31, C34, D8, R28: moved to F.Cu
- J15: value nRF debug -> STM Debug
- SW1: value SW_MEC_5G -> SW_Push; footprint Button_Switch_SMD:SW_Push_1P1T_NO_CK_KSC7xxJ -> Library:BTN_CUSTOM
- U1: footprint Package_TO_SOT_SMD:SOT-23-5 -> MCP73831T-2ACI_OT:SOT95P280X145-5N; moved to B.Cu
- moved D1 104.7 mm to (132.5, 58.6), turned to 90 degrees
- moved R13 96.1 mm to (119.0, 65.0), turned to -90 degrees
- moved J15 94.1 mm to (147.2, 60.0), turned to 90 degrees
- moved J13 85.4 mm to (157.3, 75.6), turned to -135 degrees
- moved R15 82.2 mm to (132.5, 107.4)
- moved L1 81.2 mm to (136.5, 71.5)
- moved R4 81.2 mm to (119.0, 75.0), turned to 180 degrees
- moved R2 81.0 mm to (138.5, 57.5), turned to 180 degrees
- moved R18 78.9 mm to (197.5, 63.5), turned to 90 degrees
- moved R3 77.5 mm to (119.0, 77.5), turned to 180 degrees
- moved U7 75.1 mm to (187.7, 74.5), turned to 90 degrees
- moved R11 68.7 mm to (144.5, 87.0), turned to -90 degrees
- moved R1 66.6 mm to (131.0, 76.5)
- moved R7 65.1 mm to (125.5, 98.5)
- moved U6 62.3 mm to (187.7, 85.0), turned to 90 degrees
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Routing:
- net /USB_DM: track 7.57 -> 133.7 mm, vias 1 -> 3
- net /GPS_RX: track 0.00 -> 76.1 mm, vias 0 -> 4
- net /USB_DP: track 3.25 -> 76.3 mm, vias 0 -> 8
- net VBUS: track 4.31 -> 67.7 mm, vias 1 -> 5
- net -BATT: track 101.3 -> 159.8 mm, vias 14 -> 42
- net /I2C_SDA: track 0.00 -> 54.5 mm, vias 0 -> 4
- net /LIGHT: track 0.00 -> 53.7 mm, vias 0 -> 2
- net +VCC_OUT: track 33.5 -> 87.2 mm, vias 10 -> 20
- net /nRST_STM: track 14.8 -> 58.5 mm, vias 1 -> 3
- net /GPS_TX: track 0.00 -> 36.8 mm
- net /BOOT0: track 0.00 -> 35.8 mm
- net /UART1_TX: track 0.00 -> 35.3 mm
- net /UART1_RX: track 0.00 -> 34.9 mm, vias 0 -> 2
- net +BATT: track 15.5 -> 49.0 mm, vias 0 -> 2
- net /TOUCH: track 0.00 -> 32.0 mm, vias 0 -> 2
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Other:
- board size 130 x 59.5 mm -> 100 x 59.5 mm

Commit message: complete PCB
Parts:
- removed C27: 100nF, Capacitor_SMD:C_1206_3216Metric_Pad1.33x1.80mm_HandSolder
- added D10: LED, LED_SMD:LED_0805_2012Metric_Pad1.15x1.40mm_HandSolder, F.Cu at (167.5, 113.5)
- added D6: LED, LED_SMD:LED_0805_2012Metric_Pad1.15x1.40mm_HandSolder, F.Cu at (178.5, 99.4)
- added D9: LED, LED_SMD:LED_0805_2012Metric_Pad1.15x1.40mm_HandSolder, F.Cu at (221.9, 96.2)
- added J4: Conn_01x03_Pin, Connector_JST:JST_EH_B3B-EH-A_1x03_P2.50mm_Vertical, F.Cu at (147.3, 113.0)
- added R17: 1k, Resistor_SMD:R_0805_2012Metric, B.Cu at (176.7, 102.8)
- added R23: 1k, Resistor_SMD:R_0805_2012Metric, F.Cu at (221.9, 94.0)
- added R24: 1k, Resistor_SMD:R_0805_2012Metric_Pad1.20x1.40mm_HandSolder, F.Cu at (165.5, 113.5)
- added R25: 470, Resistor_SMD:R_0805_2012Metric_Pad1.20x1.40mm_HandSolder, F.Cu at (213.5, 112.0)
- added R27: 470, Resistor_SMD:R_0805_2012Metric_Pad1.20x1.40mm_HandSolder, F.Cu at (215.0, 114.0)
- C10, C14, C15, C20, C21, C23, C26, C28, C29, C3, C30, C31, C7, C8, C9: footprint Capacitor_SMD:C_1206_3216Metric_Pad1.33x1.80mm_HandSolder -> Capacitor_SMD:C_0805_2012Metric_Pad1.18x1.45mm_HandSolder
- C11, D4, D7, D8, Q1, Q2, Q3, R10, R11, R12, R18, R21, R28, R7, R9, U10, U12, U2, U3, U5, U6, U7, U8, Y1, Y2: moved to B.Cu
- C12, C13, C22, C24: footprint Capacitor_SMD:C_1206_3216Metric_Pad1.33x1.80mm_HandSolder -> Capacitor_SMD:C_0805_2012Metric_Pad1.18x1.45mm_HandSolder; moved to F.Cu
- C16, C17, C18, C19, C32, C34, C4, C5, C6: footprint Capacitor_SMD:C_1206_3216Metric_Pad1.33x1.80mm_HandSolder -> Capacitor_SMD:C_0805_2012Metric_Pad1.18x1.45mm_HandSolder; moved to B.Cu
- D1: footprint Diode_SMD:D_0805_2012Metric -> Diode_SMD:D_SOD-323F
- D2: footprint Diode_SMD:D_SOD-523 -> Diode_SMD:D_SOD-323F
- J13: value Conn_01x04_Socket -> Conn_01x05_Socket; footprint Connector_Molex:Molex_MicroClasp_55935-0410_1x04_P2.00mm_Horizontal -> Connector_Hirose:Hirose_DF52-5S-0.8H_1x05-1MP_P0.80mm_Horizontal
- J3: footprint Connector_USB:USB_C_Receptacle_Amphenol_12401548E4-2A -> Connector_USB:USB_C_Receptacle_GCT_USB4085
- R1, R13, R6, U1: moved to F.Cu
- R22: footprint Capacitor_SMD:C_0805_2012Metric_Pad1.18x1.45mm_HandSolder -> Resistor_SMD:R_0805_2012Metric_Pad1.20x1.40mm_HandSolder; moved to B.Cu
- SW1: footprint Library:BTN_CUSTOM -> Button_Switch_SMD:SW_SPST_CK_RS282G05A3
- moved U9 133.2 mm to (241.5, 106.5)
- moved C20 124.0 mm to (230.3, 102.8), turned to 90 degrees
- moved Q4 122.9 mm to (226.9, 96.5), turned to 0 degrees
- moved R14 118.0 mm to (227.0, 101.5), turned to 180 degrees
- moved D5 103.4 mm to (221.3, 102.1), turned to 90 degrees
- moved R13 88.4 mm to (200.7, 98.8), turned to 90 degrees
- moved R15 85.2 mm to (217.5, 101.3)
- moved H1 76.4 mm to (249.3, 94.0)
- moved SW1 73.3 mm to (213.5, 119.0), turned to 180 degrees
- moved H2 70.7 mm to (249.8, 119.2)
- moved J15 69.5 mm to (184.8, 118.5), turned to -90 degrees
- moved U12 68.8 mm to (206.0, 119.0), turned to 180 degrees
- moved C21 60.1 mm to (211.5, 109.3), turned to 45 degrees
- moved J12 59.5 mm to (222.5, 118.5), turned to 0 degrees
- moved L1 59.0 mm to (173.5, 117.5), turned to 180 degrees
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Connections:
- C1 pad 2: -BATT -> GND
- C10 pad 2: -BATT -> GND
- C11 pad 2: -BATT -> GND
- C12 pad 2: -BATT -> GND
- C13 pad 2: -BATT -> GND
- C14 pad 2: -BATT -> GND
- C15 pad 2: -BATT -> GND
- C16 pad 2: -BATT -> GND
- C17 pad 2: -BATT -> GND
- C18 pad 2: -BATT -> GND
- C19 pad 2: -BATT -> GND
- C2 pad 2: -BATT -> GND
- C20 pad 2: -BATT -> GND
- C21 pad 2: -BATT -> GND
- C22 pad 2: -BATT -> GND
- C23 pad 2: -BATT -> GND
- C24 pad 2: -BATT -> GND
- C28 pad 2: -BATT -> GND
- C30 pad 2: -BATT -> GND
- C31 pad 2: -BATT -> GND
- C34 pad 2: -BATT -> GND
- C4 pad 2: -BATT -> GND
- C5 pad 2: -BATT -> GND
- C6 pad 2: -BATT -> GND
- C7 pad 2: -BATT -> GND
- C8 pad 2: -BATT -> GND
- C9 pad 2: -BATT -> GND
- D2 pad 1: -BATT -> GND
- D5 pad 1: -BATT -> GND
- E1 pad 1: -BATT -> GND
- E1 pad 12: -BATT -> GND
- E1 pad 20: unconnected-(E1-P0.07-Pad20) -> /I2C_SCL
- E1 pad 21: unconnected-(E1-P0.08-Pad21) -> /I2C_SDA
- E1 pad 24: -BATT -> GND
- E1 pad 33: unconnected-(E1-P0.19-Pad33) -> /GPS_SLEEP
- E1 pad 34: unconnected-(E1-P0.20-Pad34) -> /MEM_SLEEP
- E1 pad 39: -BATT -> GND
- E1 pad 5: unconnected-(E1-P0.28-Pad5) -> /TOUCH
- E1 pad 7: unconnected-(E1-P0.30-Pad7) -> Net-(D6-A)
- H1 pad 1: -BATT -> GND
- H2 pad 1: -BATT -> GND
- H3 pad 1: -BATT -> GND
- H4 pad 1: -BATT -> GND
- J1 pad 3: -BATT -> GND
- J1 pad 5: -BATT -> GND
- J1 pad 6: -BATT -> GND
- J1 pad 8: -BATT -> GND
- J1 pad 9: -BATT -> GND
- J11 pad 5: -BATT -> GND
- J15 pad 3: -BATT -> GND
- J15 pad 5: -BATT -> GND
- J15 pad 6: -BATT -> GND
- J15 pad 8: -BATT -> GND
- J15 pad 9: -BATT -> GND
- J3 pad A1: -BATT -> GND
- J3 pad A12: -BATT -> GND
- J3 pad B1: -BATT -> GND
- J3 pad B12: -BATT -> GND
- J5 pad 1: -BATT -> GND
- J5 pad 3: -BATT -> GND
- J6 pad 1: -BATT -> GND
- J6 pad 3: -BATT -> GND
- Q1 pad 6: -BATT -> GND
- Q1 pad 7: -BATT -> GND
- Q3 pad 2: /GPIO_SLEEP -> /MEM_SLEEP
- Q4 pad 2: /GPIO_SLEEP -> /GPS_SLEEP
- R1 pad 2: -BATT -> GND
- R11 pad 2: -BATT -> GND
- R13 pad 2: /GPIO_SLEEP -> /GPS_SLEEP
- R16 pad 2: -BATT -> GND
- R18 pad 1: -BATT -> GND
- R22 pad 2: -BATT -> GND
- R26 pad 2: /GPIO_SLEEP -> /MEM_SLEEP
- R4 pad 1: -BATT -> GND
- R5 pad 2: -BATT -> GND
- R6 pad 2: -BATT -> GND
- R7 pad 2: -BATT -> GND
- SW1 pad 1: -BATT -> GND
- U1 pad 2: -BATT -> GND
- U10 pad 1: -BATT -> GND
- U10 pad 6: -BATT -> GND
- U10 pad 9: -BATT -> GND
- U11 pad 3: -BATT -> GND
- U12 pad 1: -BATT -> GND
- U3 pad 13: -BATT -> GND
- U3 pad 15: -BATT -> GND
- U3 pad 2: -BATT -> GND
- U4 pad 17: /TOUCH -> unconnected-(U4-PA2-Pad17)
- U4 pad 19: /BAT_ALERT -> unconnected-(U4-PA4-Pad19)
- U4 pad 20: unconnected-(U4-PA5-Pad20) -> /STAT_LED
- U4 pad 32: -BATT -> GND
- U4 pad 34: -BATT -> Net-(U4-OSC_OUT)
- U4 pad 35: -BATT -> Net-(U4-OSC_IN)
- U4 pad 42: -BATT -> GND
- U4 pad 69: -BATT -> GND
- U5 pad 4: -BATT -> GND
- U6 pad 2: -BATT -> GND
- U7 pad 2: -BATT -> GND
- U8 pad 5: -BATT -> GND
- U9 pad 10: /GPS_RX -> Net-(U9-RX)
- U9 pad 12: -BATT -> GND
- U9 pad 14: /I2C_SCL -> unconnected-(U9-RX1/I2C_SCL-Pad14)
- U9 pad 15: /I2C_SDA -> unconnected-(U9-TX1/I2C_SDA-Pad15)
- U9 pad 19: -BATT -> GND
- U9 pad 3: -BATT -> GND
- U9 pad 8: -BATT -> GND
- U9 pad 9: /GPS_TX -> Net-(U9-TX)
- Y1 pad 1: -BATT -> Net-(U4-OSC_OUT)
- Y1 pad 2: -BATT -> Net-(U4-OSC_IN)
Routing:
- net GND: track 0.00 -> 137.4 mm, vias 0 -> 70
- net -BATT: track 159.8 -> 51.4 mm, vias 42 -> 0
- net /USB_DM: track 133.7 -> 63.3 mm, vias 3 -> 0
- net /GPS_RX: track 76.1 -> 8.30 mm, vias 4 -> 0
- net /I2C_SCL: track 0.00 -> 53.2 mm, vias 0 -> 4
- net /BAT_ALERT: track 0.00 -> 50.1 mm, vias 0 -> 3
- net /GPS_SLEEP: track 0.00 -> 47.2 mm, vias 0 -> 1
- net /SPI1_SCK: track 0.00 -> 39.6 mm, vias 0 -> 2
- net /LIGHT: track 53.7 -> 18.1 mm, vias 2 -> 3
- net +VCC_OUT: track 87.2 -> 120.2 mm, vias 20 -> 26
- net /GPS_TX: track 36.8 -> 4.57 mm
- net VBUS: track 67.7 -> 39.2 mm, vias 5 -> 2
- net /MEM_SLEEP: track 0.00 -> 28.2 mm, vias 0 -> 2
- net /OSC32_IN: track 0.00 -> 28.0 mm, vias 0 -> 5
- net /UART1_TX: track 35.3 -> 9.23 mm
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- added copper zone on F.Cu, net GND
- added copper zone on In1.Cu, net GND
- removed copper zone on B.Cu, net +VCC_OUT
- removed copper zone on In1.Cu, net -BATT
Other:
- board size 100 x 59.5 mm -> 110 x 30.5 mm
- board text added: "BATT IN"
- board text added: "Power Out"
- board text removed: "LDR"
- board text removed: "Touch Sensors"

Commit message: implement some feedback
Parts:
- removed R22: 1M, Resistor_SMD:R_0805_2012Metric_Pad1.20x1.40mm_HandSolder
- moved D1 6.45 mm to (152.9, 101.6)
- moved C34 3.85 mm to (211.3, 106.4)
- moved H4 0.30 mm to (171.3, 102.5)
Connections:
- H1 pad 1: GND -> unconnected-(H1-Pad1)
- H2 pad 1: GND -> unconnected-(H2-Pad1)
- H3 pad 1: GND -> unconnected-(H3-Pad1)
- H4 pad 1: GND -> unconnected-(H4-Pad1)
- J3 pad S1: Net-(J3-SHIELD) -> GND
- U3 pad 13: GND -> Net-(U3-EN)
- U4 pad 13: unconnected-(U4-VREF+-Pad13) -> +VCC_OUT
Routing:
- net Net-(J3-SHIELD): track 27.1 -> 0.00 mm
- net /OSC32_IN: track 28.0 -> 51.8 mm
- net GND: track 137.4 -> 157.6 mm, vias 70 -> 69
- net /MEM_SLEEP: track 28.2 -> 20.0 mm, vias 2 -> 1
- net Net-(D1-A): track 1.86 -> 9.75 mm
- net Net-(D2-A2): track 7.06 -> 10.9 mm
- net STAT: track 2.08 -> 5.00 mm
- net +VCC_OUT: track 120.2 -> 123.0 mm, vias 26 -> 27
- net VBUS: track 39.2 -> 41.9 mm
- net /USB_DM: track 63.3 -> 61.0 mm
- net /I2C_SDA: track 38.9 -> 36.8 mm
- net /TOUCH_B: track 24.8 -> 23.1 mm
- net /USB_DP: track 60.4 -> 58.8 mm
- net /GPS_SLEEP: track 47.2 -> 45.7 mm
- net +BATT: track 69.2 -> 67.8 mm, vias 4 -> 2
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Other:
- board text added: "C12"
- board text added: "U1"
