File: FitLensPCB.kicad_sch (KiCad schematic)
At the start: 62 parts, among them J1 Debugging Antenna, J2 Conn_01x02_Pin, J3 USB_C_Receptacle_USB2.0_16P, J4 Conn_01x03_Pin, Q1 FS8205A, Q2 AO3401A, SW1 SW_MEC_5G, U1 MCP73831-2-OT, U2 DW01A, U3 TPS63020DSJR, U4 STM32WB55RGVx, U5 MX25L3233FM1, U6 AT42QT1010-TSHR

Commit message: complete most of schematic
Parts:
- added C26, C29: C, Capacitor_SMD:C_0603_1608Metric_Pad1.08x0.95mm_HandSolder, symbol Device:C
- added C27, C28, C30, C31: 100nF, Capacitor_SMD:C_0603_1608Metric_Pad1.08x0.95mm_HandSolder, symbol Device:C
- added C32: 100nF, symbol Device:C_US
- added D5: 1N4148W, Diode_SMD:D_SOD-123, symbol Diode:1N4148W
- added D6: LED, LED_SMD:LED_0603_1608Metric_Pad1.05x0.95mm_HandSolder, symbol Device:LED
- added J10, J7, J8, J9: 1x1, Connector_PinHeader_2.54mm:PinHeader_1x01_P2.54mm_Vertical, symbol Connector:Conn_01x01_Pin
- added J11: Conn_Coaxial, Connector_Coaxial:U.FL_Hirose_U.FL-R-SMT-1_Vertical, symbol Connector:Conn_Coaxial
- added J12: Conn_01x02_Pin, Connector_JST:JST_PH_S2B-PH-K_1x02_P2.00mm_Horizontal, symbol Connector:Conn_01x02_Pin
- added J13: Conn_01x04_Socket, Connector_Molex:Molex_MicroClasp_55935-0410_1x04_P2.00mm_Horizontal, symbol Connector:Conn_01x04_Socket
- added J5, J6: Conn_01x03_Pin, Connector_JST:JST_XH_S3B-XH-A-1_1x03_P2.50mm_Horizontal, symbol Connector:Conn_01x03_Pin
- added R12, R9: R_S, Resistor_SMD:R_0603_1608Metric_Pad0.98x0.95mm_HandSolder, symbol Device:R_US
- added R13, R15: 10k, symbol Device:R_US
- added R14: 1k, symbol Device:R_US
- added R16, R17: 470, symbol Device:R_US
- added R18: R_LDR, Resistor_SMD:R_0201_0603Metric_Pad0.64x0.40mm_HandSolder, symbol Device:R_US
- added R19, R20: 47k, Resistor_SMD:R_0201_0603Metric_Pad0.64x0.40mm_HandSolder, symbol Device:R_US
- added U10: MAX17048G_T10, MAX17048G_T10:SON50P200X200X80-9N, symbol MAX17048G_T10:MAX17048G_T10
- added U7: AT42QT1010-TSHR, Package_TO_SOT_SMD:SOT-23-6, symbol Sensor_Touch:AT42QT1010-TSHR
- added U8: 74AHC1G08, Package_TO_SOT_SMD:SOT-23-5_HandSoldering, symbol 74xGxx:74AHC1G08
- added U9: 5186, PA1616D:CD-PA1616D_ADA, symbol PA1616D:5186
Connections:
- net GND is gone; now on net -BATT: C1.2, C10.2, C11.2, C12.2, C13.2, C14.2, C15.2, C16.2, C17.2, C18.2, C19.2, C2.2, C22.1, C23.1, C24.2, C25.2, C4.2, C5.2, C6.2, C7.2, C8.2, C9.2, D2.1 (A1), FL1.2, FL1.2_1, H1.1, H2.1, H3.1, H4.1, J1.2 (Ext), J3.A1 (GND), J3.A12 (GND), J3.B1 (GND), J3.B12 (GND), J3.S1 (SHIELD), J4.1 (Pin_1), Q1.6, Q1.7, R1.2, R11.2, R4.1, R5.2, R6.2, R7.2, SW1.1 (A), SW1.2 (A), U1.2 (V_{SS}), U3.13 (PS/SYNC), U3.15 (PGND), U3.2 (GND), U4.32 (VSSRF), U4.42 (VSSSMPS), U4.69 (VSS), U5.4 (GND), U6.2 (VSS)
- net +BATT: now also C32.1, U10.2 (CELL)
- net +VCC_OUT: now also C27.1, C28.1, C30.1, C31.1, J12.2 (Pin_2), R13.1, R15.1, R19.2, R20.2, U10.3 (VDD), U7.5 (VDD), U8.3 (GND), U9.1 (VCC), U9.4 (VBACKUP)
- net -BATT: now also C27.2, C28.2, C30.2, C31.2, C32.2, J11.2 (Ext), J5.1 (Pin_1), J5.3 (Pin_3), J6.1 (Pin_1), J6.3 (Pin_3), R14.2, R18.1, U10.1 (CTG), U10.4 (GND), U10.6 (QSTRT), U10.9 (EP), U7.2 (VSS), U8.5 (VCC), U9.12 (GND), U9.19 (GND), U9.3 (GND), U9.8 (GND)
- net TOUCH_A: now reaches U6.1 (OUT)
- net TOUCH_A: now also J9.1 (Pin_1), U8.2
- net at U6.3 (SNSK): now also C26.1, R9.1
- net at U6.4 (SNS): now also C26.2
- net QSPI_NCS: now reaches U5.1 (~{CS})
- net QSPI_NCS: now also U4.29 (PB11)
- net QSPI_SIO1: now reaches U5.2 (SO/SIO1)
- net QSPI_SIO2: now reaches U5.3 (~{WP}/SIO2)
- net QSPI_SIO0: now reaches U5.5 (SI/SIO0)
- net QSPI_SCK: now reaches U5.6 (SCLK)
- net QSPI_SCK: now also U4.18 (PA3)
- net QSPI_SIO3: now reaches U5.7 (~{HOLD}/SIO3)
- net QSPI_IO3: now reaches U4.10 (PC1)
- net QSPI_IO3: now also U4.21 (PA6)
- net LIGHT: now reaches U4.15 (PA0)
- net LIGHT: now also J12.1 (Pin_1), R18.2
- net SPI1_SCK: now reaches U4.16 (PA1)
- net TOUCH: now reaches U4.17 (PA2)
- net TOUCH: now also J7.1 (Pin_1)
- net QSPI_IO2: now reaches U4.22 (PA7)
- net QSPI_IO2: now also U4.9 (PC0)
- net BAT_ALERT: now reaches U4.23 (PA8)
- net BAT_ALERT: now also U10.5 (~{ALERT})
- net I2C_SCL: now reaches U4.24 (PA9)
- net I2C_SCL: now also R19.1, U9.14 (RX1(I2C_SCL))
- net I2C_SDA: now reaches U4.51 (PA10)
- net I2C_SDA: now also R20.1, U10.8 (SDA), U9.15 (TX1(I2C_SDA))
- net SPI1_CS: now reaches U4.57 (PA15)
- net SPI1_CS: now also J13.4 (Pin_4)
- net SPI1_DC: now reaches U4.58 (PC10)
- net SPI1_DC: now also J13.1 (Pin_1)
- net QSPI_IO1: now reaches U4.6 (PB8)
- net SPI1_RST: now reaches U4.60 (PC12)
- net SPI1_RST: now also J13.2 (Pin_2)
- net SPI1_MOSI: now reaches U4.65 (PB5)
- net SPI1_MOSI: now also J13.3 (Pin_3)
- net UART1_TX: now reaches U4.66 (PB6)
- net UART1_TX: now also D5.1 (K)
- net UART1_RX: now reaches U4.67 (PB7)
- net UART1_RX: now also R17.2
- net QSPI_IO0: now reaches U4.7 (PB9)
- new net: J6.2 (Pin_2), R12.2
- new net: J11.1 (In), U9.11 (EX_ANT)
- new net: D6.1 (K), R14.1
- new net: R17.1, U9.9 (TX0)
- new net: C29.1, R12.1, U7.3 (SNSK)
- new net: C29.2, U7.4 (SNS)
- new net: D5.2 (A), R16.1
- new net: R13.2, R16.2, U9.10 (RX0)
- new net: J5.2 (Pin_2), R9.2
- new net: D6.2 (A), U9.5 (3D-FIX)
- new net GPS_NRST: R15.2, U9.2 (NRESET)
- new net I2C1_SCL: U10.7 (SCL)
- new net TOUCH_AND: J8.1 (Pin_1), U8.4
- new net TOUCH_B: J10.1 (Pin_1), U7.1 (OUT), U8.1
Other:
- note added: "Display Header"
- note added: "Fuel Gauge IC"
- note added: "GPS Module"
- note added: "Microcontroller"
- note added: "R1 = R2 * (Vout / FB - 1) [1] - page 15 Vout = (FB * (R1 + R2)) / R2 FB = 500mV Vmin = (500mV * (1,1MOhm + 100KOhm + 120KOhm)) ------------------------------ 120KOhm + 100KOhm = 3V Vmax = (500mV * (1,1MOhm + 100KOhm + 120KOhm)) ----------------------------- 120KOhm = 5,5V"
- note added: "Touch Sensor A"
- note added: "Touch Sensor B"
- note added: "Touch sensor headers"
- note added: "Use internal pull-up resistor on PA4 for BAT_ALERT signal since it's active low and there is no space for an external pull-up"
- note added: "headers to all be placed at 2.54mm from each other in layout"
- note added: "if MOSFET for VCC (for sleep mode), connect VBACKUP to power immediately"
- note added: "touch sensor AND Gate"
- note removed: "R1 = R2 * (Vout / FB - 1) [1] - page 15 Vout = (FB * (R1 + R2)) / R2 FB = 500mV Vmin = (500mV * (1,1MOhm + 100KOhm + 120KOhm)) / 120KOhm + 100KOhm = 3V Vmax = (500mV * (1,1MOhm + 100KOhm + 120KOhm)) / 120KOhm = 5,5V"
- note removed: "Touch Sensor"
- moved on the sheet: C12, C13, C14, C15, C16, C17, C18, C19, C20, C21, C22, C23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

Commit message: I dont even know anymore
Parts:
- removed C21, C22, C23, C25: 0pF, Capacitor_SMD:C_0402_1005Metric_Pad0.74x0.62mm_HandSolder, symbol Device:C
- removed C24: 1.2pF, Capacitor_SMD:C_0402_1005Metric_Pad0.74x0.62mm_HandSolder, symbol Device:C
- removed C30, C31: 100nF, Capacitor_SMD:C_0603_1608Metric_Pad1.08x0.95mm_HandSolder, symbol Device:C
- removed D5: 1N4148W, Diode_SMD:D_SOD-123, symbol Diode:1N4148W
- removed D6: LED, LED_SMD:LED_0603_1608Metric_Pad1.05x0.95mm_HandSolder, symbol Device:LED
- removed FL1: LFB182G45CGFD436, LFB182G45CGFD436:FIL_LFB182G45CGFD436, symbol LFB182G45CGFD436:LFB182G45CGFD436
- removed J1: Debugging Antenna, Connector_Coaxial:SMA_Amphenol_132134-10_Vertical, symbol Connector:Conn_Coaxial_Small
- removed J11: Conn_Coaxial, Connector_Coaxial:U.FL_Hirose_U.FL-R-SMT-1_Vertical, symbol Connector:Conn_Coaxial
- removed L2: 2.7nH, Inductor_SMD:L_0201_0603Metric_Pad0.64x0.40mm_HandSolder, symbol Device:L
- removed L3: 0H, Inductor_SMD:L_0402_1005Metric_Pad0.77x0.64mm_HandSolder, symbol Device:L
- removed L4: L, Inductor_SMD:L_0402_1005Metric_Pad0.77x0.64mm_HandSolder, symbol Device:L
- removed R15: 10k, symbol Device:R_US
- removed R16, R17: 470, symbol Device:R_US
- removed R8: 10k, Resistor_SMD:R_0603_1608Metric_Pad0.98x0.95mm_HandSolder, symbol Device:R
- removed RV1: 100K, Potentiometer_THT:Potentiometer_Bourns_3296W_Vertical, symbol Device:R_Potentiometer
- removed U9: 5186, PA1616D:CD-PA1616D_ADA, symbol PA1616D:5186
- added D5: LED, LED_SMD:LED_0805_2012Metric, symbol Device:LED
- added D7, D8: SB120, Diode_THT:D_DO-41_SOD81_P10.16mm_Horizontal, symbol Diode:SB120
- added E1: MDBT42Q-512KV2, MDBT42Q-512KV2:RAYTAC_MDBT42Q-512KV2, symbol MDBT42Q-512KV2:MDBT42Q-512KV2
- added J1, J15: nRF debug, Connector_PinHeader_1.27mm:PinHeader_2x05_P1.27mm_Horizontal, symbol Connector:Conn_ARM_JTAG_SWD_10
- added J14: Conn_Coaxial, Connector_Coaxial:U.FL_Hirose_U.FL-R-SMT-1_Vertical, symbol Connector:Conn_Coaxial
- added Q3, Q4: PMOS, symbol Simulation_SPICE:PMOS
- added R21: 25M, Resistor_SMD:R_0805_2012Metric_Pad1.20x1.40mm_HandSolder, symbol Device:R_US
- added R22: 1M, symbol Device:R_US
- added R26, R28, R8: 10k, symbol Device:R_US
- added U11: TPD2EUSB30, Package_TO_SOT_SMD:Texas_DRT-3, symbol Power_Protection:TPD2EUSB30
- added U9: CD-PA1616D, CD-PA1616D:XCVR_CD-PA1616D, symbol CD-PA1616D:CD-PA1616D
- added Y1: 32mHz, Crystal:Crystal_SMD_0603-2Pin_6.0x3.5mm_HandSoldering, symbol Device:Crystal
- added Y2: 32.768kHz, Crystal:Crystal_SMD_FOX_FE-2Pin_7.5x5.0mm_HandSoldering, symbol Device:Crystal
- C18: value 0.8pF -> C; footprint Capacitor_SMD:C_0504_1310Metric_Pad0.83x1.28mm_HandSolder -> Capacitor_SMD:C_01005_0402Metric_Pad0.57x0.30mm_HandSolder
- C19: value 0.3pF -> C; footprint Capacitor_SMD:C_0504_1310Metric_Pad0.83x1.28mm_HandSolder -> Capacitor_SMD:C_01005_0402Metric_Pad0.57x0.30mm_HandSolder
- C20: value 10nF -> 100nF; footprint Capacitor_SMD:C_0402_1005Metric_Pad0.74x0.62mm_HandSolder -> Capacitor_SMD:C_0603_1608Metric_Pad1.08x0.95mm_HandSolder
- J5: value Conn_01x03_Pin -> Conn_Pin
- R10: value 1,1M -> 56k; footprint Resistor_SMD:R_0603_1608Metric -> Resistor_SMD:R_0805_1608Metric
- R11: value 120K -> 10k; footprint Resistor_SMD:R_0603_1608Metric -> Resistor_SMD:R_0805_1608Metric
- R14: value 1k -> R_US; footprint (none) -> Resistor_SMD:R_0805_2012Metric_Pad1.20x1.40mm_HandSolder
Connections:
- net +VCC_OUT: now also C20.1, U4.1 (VBAT), E1.11 (VDD), J1.1 (VTref), J15.1 (VTref), Q3.1 (D), Q4.1 (D), R26.1, R28.1, R8.1, U9.4 (VBACKUP); no longer U5.8 (VCC)
- net -BATT: now also C20.2, U4.34 (OSC_OUT), U4.35 (OSC_IN), D5.1 (K), E1.1 (GND), E1.12 (GND), E1.24 (GND), E1.39 (GND), J1.3 (GND), J1.5 (GND), J1.6 (SWO/TDO), J1.8 (NC/TDI), J1.9 (GNDDetect), J14.2 (Ext), J15.3 (GND), J15.5 (GND), J15.6 (SWO/TDO), J15.8 (NC/TDI), J15.9 (GNDDetect), R22.2, U11.3 (GND), U9.12 (GND), U9.19 (GND), U9.3 (GND), U9.8 (GND), Y1.1, Y1.2; no longer J3.S1 (SHIELD), R14.2
- net BAT_ALERT: now also U4.19 (PA4)
- net FB: now also R10.2, R11.1
- net I2C_SCL: now also U9.14 (RX1/I2C_SCL)
- net I2C_SDA: now also U9.15 (TX1/I2C_SDA)
- net RF_LINE: now also J14.1 (In); no longer C18.1
- net USB_DM: now also U11.2 (D-)
- net USB_DP: now also U11.1 (D+)
- net at SW1.3 (B), SW1.4 (B): now also D7.1 (K), D8.1 (K); no longer U4.8 (NRST)
- net GPS_FIX: now reaches R14.1
- net GPS_FIX: now also U9.5 (3D-FIX)
- net GPIO_SLEEP: now reaches R13.2
- net GPIO_SLEEP: now also Q3.2 (G), Q4.2 (G), R26.2
- net OSC32_IN: now reaches C19.1
- net OSC32_IN: now also U4.2 (PC13), Y2.1
- net OSC32_OUT: now reaches U4.3 (PC14)
- net OSC32_OUT: now also R21.2
- net SWCLK_STM: now reaches U4.54 (PA13)
- net SWCLK_STM: now also J15.4 (SWCLK/TCK)
- net SWDIO_STM: now reaches U4.56 (PA14)
- net SWDIO_STM: now also J15.2 (SWDIO/TMS)
- new net: Q4.3 (S), U9.1 (VCC)
- new net: U9.16 (NC), U9.17 (NC), U9.18 (NC), U9.20 (NC), U9.6 (NC), U9.7 (NC)
- new net: J3.S1 (SHIELD), R22.1
- new net: C18.1, R21.1, Y2.2
- new net: D5.2 (A), R14.2
- new net: Q3.3 (S), U5.8 (VCC)
- new net GPS_1PPS: U9.13 (1PPS)
- new net GPS_RX: U9.10 (RX)
- new net GPS_TX: U9.9 (TX)
- new net SWCLK_nRF: E1.36 (SWDCLK), J1.4 (SWCLK/TCK)
- new net SWDIO_nRF: E1.37 (SWDIO), J1.2 (SWDIO/TMS)
- new net nRST_GPS: U9.2 (~{RESET})
- new net nRST_STM: D8.2 (A), J15.10 (~{RESET}), R28.2, U4.8 (NRST)
- new net nRST_nRF: D7.2 (A), E1.35 (P0.21/RESET), J1.10 (~{RESET}), R8.2
Other:
- note added: "Debug Headers"
- note added: "FB = 500mV"
- note added: "LSE Oscillator Circuit"
- note added: "Power LED on 3.3V"
- note added: "Raytac BLE Module"
- note added: "Static protection chip add here"
- note added: "VCC_OUT = FB * (1 + R1/R2) = 500mV * (1 + 56k / 10k) = 3.3V"
- note added: "add debouncing"
- note added: "nRST Circuitry"
- note added: "reverse current diodes"
- note added: "u.fl antenna (place as close to RF pin as possible)"
- note removed: "Antenna Impedance Matching Circuit"
- note removed: "Debugging antenna line. C & L value undetermined and depend on debugging antenna used."
- note removed: "R1"
- note removed: "R1 = R2 * (Vout / FB - 1) [1] - page 15 Vout = (FB * (R1 + R2)) / R2 FB = 500mV Vmin = (500mV * (1,1MOhm + 100KOhm + 120KOhm)) ------------------------------ 120KOhm + 100KOhm = 3V Vmax = (500mV * (1,1MOhm + 100KOhm + 120KOhm)) ----------------------------- 120KOhm = 5,5V"
- note removed: "R2"
- note removed: "if MOSFET for VCC (for sleep mode), connect VBACKUP to power immediately"
- moved on the sheet: SW1, U5

Commit message: complete schematic allegedly
Parts:
- added C21, C22, C23, C25: 100nF, Capacitor_SMD:C_0603_1608Metric_Pad1.08x0.95mm_HandSolder, symbol Device:C
- added C24: 10uF, Capacitor_SMD:C_0603_1608Metric_Pad1.08x0.95mm_HandSolder, symbol Device:C
- added J11: Conn_01x05_Pin, Connector_Hirose:Hirose_DF13-05P-1.25DS_1x05_P1.25mm_Horizontal, symbol Connector:Conn_01x05_Pin
- added R15, R16: 10k, Resistor_SMD:R_0805_2012Metric_Pad1.20x1.40mm_HandSolder, symbol Device:R_US
- added U12: MAX6816, Package_TO_SOT_SMD:SOT-143, symbol Interface:MAX6816
- R1, R2, R3, R4, R5, R6, R7: footprint Resistor_SMD:R_0603_1608Metric -> Resistor_SMD:R_0805_2012Metric_Pad1.20x1.40mm_HandSolder
- R10, R11: footprint Resistor_SMD:R_0805_1608Metric -> Resistor_SMD:R_0805_2012Metric_Pad1.20x1.40mm_HandSolder
- R12, R9: footprint Resistor_SMD:R_0603_1608Metric_Pad0.98x0.95mm_HandSolder -> Resistor_SMD:R_0805_2012Metric_Pad1.20x1.40mm_HandSolder
- R13, R26, R28, R8: footprint (none) -> Resistor_SMD:R_0805_2012Metric_Pad1.20x1.40mm_HandSolder
- R14: value R_US -> 1k
- R18, R19, R20: footprint Resistor_SMD:R_0201_0603Metric_Pad0.64x0.40mm_HandSolder -> Resistor_SMD:R_0805_2012Metric_Pad1.20x1.40mm_HandSolder
Connections:
- net +VCC_OUT: now also C21.1, C22.1, C23.1, C24.1, C25.1, J11.1 (Pin_1), R15.2, U12.4 (VCC)
- net -BATT: now also C21.2, C22.2, C23.2, C24.2, C25.2, J11.5 (Pin_5), R16.2, U12.1 (GND)
- net BAT_ALERT: now also R15.1
- net GPS_RX: now also U4.10 (PC1)
- net GPS_TX: now also U4.9 (PC0)
- net QSPI_IO2: no longer U4.9 (PC0)
- net QSPI_IO3: no longer U4.10 (PC1)
- net UART1_RX: now also J11.4 (Pin_4)
- net UART1_TX: now also J11.3 (Pin_3)
- net at D7.1 (K), D8.1 (K): now also U12.3 (OUT); no longer SW1.3 (B), SW1.4 (B)
- net BOOT0: now reaches U4.5 (PH3)
- net BOOT0: now also J11.2 (Pin_2), R16.1
- new net: SW1.3 (B), SW1.4 (B), U12.2 (IN)
Other:
- note added: "UART1 Header (can program STM32 if necessary)"
- note removed: "Static protection chip add here"
- note removed: "Use internal pull-up resistor on PA4 for BAT_ALERT signal since it's active low and there is no space for an external pull-up"
- note removed: "add debouncing"
- note removed: "reverse current diodes"
- moved on the sheet: C18, C19, C20, D5, D7, D8, E1, J14, Q4, R13, R14, R19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

Commit message: screw this
Parts:
- removed C25: 100nF, Capacitor_SMD:C_0603_1608Metric_Pad1.08x0.95mm_HandSolder, symbol Device:C
- removed J14: Conn_Coaxial, Connector_Coaxial:U.FL_Hirose_U.FL-R-SMT-1_Vertical, symbol Connector:Conn_Coaxial
- added C30: 100nF, Capacitor_SMD:C_1206_3216Metric_Pad1.33x1.80mm_HandSolder, symbol Device:C
- added C31: 2.2uF, Capacitor_SMD:C_1206_3216Metric_Pad1.33x1.80mm_HandSolder, symbol Device:C
- added C34: 4.7uF, Capacitor_SMD:C_1206_3216Metric_Pad1.33x1.80mm_HandSolder, symbol Device:C
- C10, C3, C4, C5, C6, C7, C8, C9: footprint Capacitor_SMD:C_0805_2012Metric -> Capacitor_SMD:C_1206_3216Metric_Pad1.33x1.80mm_HandSolder
- C12, C13, C14, C15, C16, C17, C20, C21, C22, C24, C26, C27, C28, C29: footprint Capacitor_SMD:C_0603_1608Metric_Pad1.08x0.95mm_HandSolder -> Capacitor_SMD:C_1206_3216Metric_Pad1.33x1.80mm_HandSolder
- C18, C19: footprint Capacitor_SMD:C_01005_0402Metric_Pad0.57x0.30mm_HandSolder -> Capacitor_SMD:C_1206_3216Metric_Pad1.33x1.80mm_HandSolder
- C23: value 100nF -> 1uF; footprint Capacitor_SMD:C_0603_1608Metric_Pad1.08x0.95mm_HandSolder -> Capacitor_SMD:C_1206_3216Metric_Pad1.33x1.80mm_HandSolder
- C32: footprint (none) -> Capacitor_SMD:C_1206_3216Metric_Pad1.33x1.80mm_HandSolder
- D7, D8: value SB120 -> SS12; footprint Diode_THT:D_DO-41_SOD81_P10.16mm_Horizontal -> Diode_SMD:D_SOD-123F
- J2: footprint Cutom_PinHeaders:PinSocket_1x02_P2.54mm_Vertical -> Connector_JST:JST_PH_B2B-PH-K_1x02_P2.00mm_Vertical
- J3: footprint (none) -> Connector_USB:USB_C_Receptacle_Amphenol_12401548E4-2A
- R22: footprint (none) -> Capacitor_SMD:C_0805_2012Metric_Pad1.18x1.45mm_HandSolder
- SW1: footprint Button_Switch_SMD:SW_MEC_5GSH9 -> Button_Switch_SMD:SW_Push_1P1T_NO_CK_KSC7xxJ
Connections:
- net I2C1_SCL is gone; now on net I2C_SCL: U10.7 (SCL)
- net +VCC_OUT: now also C30.1, C31.1, C34.1
- net -BATT: now also C30.2, C31.2, C34.2
Other:
- note added: "VDD Decoupling Caps"
- note added: "VDDA Decoupling Caps"
- note added: "VDDRF Decoupling Caps"
- note removed: "u.fl antenna (place as close to RF pin as possible)"
- moved on the sheet: C12, C13, C22

Commit message: lol
Parts:
- removed C15, C27: 100nF, Capacitor_SMD:C_1206_3216Metric_Pad1.33x1.80mm_HandSolder, symbol Device:C
- removed SW1: SW_MEC_5G, Button_Switch_SMD:SW_Push_1P1T_NO_CK_KSC7xxJ, symbol Switch:SW_MEC_5G
- added SW1: SW_Push, Library:BTN_CUSTOM, symbol Switch:SW_Push
- J15: value nRF debug -> STM Debug
- Q1: footprint footprints:SOP65P640X120-8N -> FS8205A:SOP65P640X120-8N
- Q3, Q4: footprint (none) -> Package_TO_SOT_SMD:SOT-723
- U1: footprint Package_TO_SOT_SMD:SOT-23-5 -> MCP73831T-2ACI_OT:SOT95P280X145-5N
- U2: footprint footprints:SOT23-6 -> DW01A:SOT95P280X145-6N
- U3: footprint footprints:IC_TPS63020DSJR -> TPS63020DSJR:IC_TPS63020DSJR
- U5: footprint (none) -> MX25L3233FM2I-08G:SOIC127P790X216-8N_MX25L3233FM2I-08G
Connections:
- net QSPI_SIO0 is gone; now on net QSPI_IO0: U5.5 (SI/SIO0)
- net QSPI_SIO1 is gone; now on net QSPI_IO1: U5.2 (SO/SIO1)
- net QSPI_SIO2 is gone; now on net QSPI_IO2: U5.3 (~{WP}/SIO2)
- net QSPI_SIO3 is gone; now on net QSPI_IO3: U5.7 (~{HOLD}/SIO3)
- net -BATT: now also SW1.1
- net at U12.2 (IN): now also SW1.2
Other:
- moved on the sheet: Q1

Commit message: complete PCB
Parts:
- added C15: 100nF, Capacitor_SMD:C_0805_2012Metric_Pad1.18x1.45mm_HandSolder, symbol Device:C
- added D10, D6, D9: LED, LED_SMD:LED_0805_2012Metric_Pad1.15x1.40mm_HandSolder, symbol Device:LED
- added R17, R23: 1k, Resistor_SMD:R_0805_2012Metric, symbol Device:R_US
- added R24: 1k, Resistor_SMD:R_0805_2012Metric_Pad1.20x1.40mm_HandSolder, symbol Device:R_US
- added R25, R27: 470, Resistor_SMD:R_0805_2012Metric_Pad1.20x1.40mm_HandSolder, symbol Device:R_US
- C10, C12, C13, C14, C16, C17, C18, C19, C20, C21, C22, C23, C24, C26, C28, C29, C3, C30, C31, C32, C34, C4, C5, C6, C7, C8, C9: footprint Capacitor_SMD:C_1206_3216Metric_Pad1.33x1.80mm_HandSolder -> Capacitor_SMD:C_0805_2012Metric_Pad1.18x1.45mm_HandSolder
- D1: footprint Diode_SMD:D_0805_2012Metric -> Diode_SMD:D_SOD-323F
- D2: footprint Diode_SMD:D_SOD-523 -> Diode_SMD:D_SOD-323F
- J13: value Conn_01x04_Socket -> Conn_01x05_Socket; footprint Connector_Molex:Molex_MicroClasp_55935-0410_1x04_P2.00mm_Horizontal -> Connector_Hirose:Hirose_DF52-5S-0.8H_1x05-1MP_P0.80mm_Horizontal; symbol Connector:Conn_01x04_Socket -> Connector:Conn_01x05_Socket
- J3: footprint Connector_USB:USB_C_Receptacle_Amphenol_12401548E4-2A -> Connector_USB:USB_C_Receptacle_GCT_USB4085
- J4: footprint Cutom_PinHeaders:PinHeader_1x03_P2.54mm_Vertical -> Connector_JST:JST_EH_B3B-EH-A_1x03_P2.50mm_Vertical
- R22: footprint Capacitor_SMD:C_0805_2012Metric_Pad1.18x1.45mm_HandSolder -> Resistor_SMD:R_0805_2012Metric_Pad1.20x1.40mm_HandSolder
- SW1: footprint Library:BTN_CUSTOM -> Button_Switch_SMD:SW_SPST_CK_RS282G05A3
Connections:
- net +VCC_OUT: now also C15.1, D10.2 (A)
- net -BATT: no longer C1.2, C10.2, C11.2, C12.2, C13.2, C14.2, C16.2, C17.2, C18.2, C19.2, C2.2, C20.2, C21.2, C22.2, C23.2, C24.2, C28.2, C30.2, C31.2, C34.2, C4.2, C5.2, C6.2, C7.2, C8.2, C9.2, D2.1 (A1), D5.1 (K), E1.1 (GND), E1.12 (GND), E1.24 (GND), E1.39 (GND), H1.1, H2.1, H3.1, H4.1, J1.3 (GND), J1.5 (GND), J1.6 (SWO/TDO), J1.8 (NC/TDI), J1.9 (GNDDetect), J11.5 (Pin_5), J15.3 (GND), J15.5 (GND), J15.6 (SWO/TDO), J15.8 (NC/TDI), J15.9 (GNDDetect), J3.A1 (GND), J3.A12 (GND), J3.B1 (GND), J3.B12 (GND), J4.1 (Pin_1), J5.1 (Pin_1), J5.3 (Pin_3), J6.1 (Pin_1), J6.3 (Pin_3), Q1.6, Q1.7, R1.2, R11.2, R16.2, R18.1, R22.2, R4.1, R5.2, R6.2, R7.2, SW1.1, U1.2 (V_{SS}), U10.1 (CTG), U10.6 (QSTRT), U10.9 (EP), U11.3 (GND), U12.1 (GND), U3.13 (PS/SYNC), U3.15 (PGND), U3.2 (GND), U4.32 (VSSRF), U4.34 (OSC_OUT), U4.35 (OSC_IN), U4.42 (VSSSMPS), U4.69 (VSS), U5.4 (GND), U6.2 (VSS), U7.2 (VSS), U8.5 (VCC), U9.12 (GND), U9.19 (GND), U9.3 (GND), U9.8 (GND), Y1.1, Y1.2
- net BAT_ALERT: no longer U4.19 (PA4)
- net GPS_RX: now also R27.1; no longer U9.10 (RX)
- net GPS_TX: now also R25.1; no longer U9.9 (TX)
- net I2C_SCL: now also E1.20 (P0.07); no longer U9.14 (RX1/I2C_SCL)
- net I2C_SDA: now also E1.21 (P0.08); no longer U9.15 (TX1/I2C_SDA)
- net SPI1_SCK: now also J13.5 (Pin_5)
- net TOUCH: now also E1.5 (P0.28); no longer U4.17 (PA2)
- net GPS_SLEEP: now reaches E1.33 (P0.19)
- net GPS_SLEEP: now also Q4.2 (G), R13.2
- net MEM_SLEEP: now reaches E1.34 (P0.20)
- net MEM_SLEEP: now also Q3.2 (G), R26.2
- net at E1.7 (P0.30): now also D6.2 (A)
- net STAT_LED: now reaches U4.20 (PA5)
- net STAT_LED: now also D9.2 (A)
- removed net GPIO_SLEEP: Q3.2 (G), Q4.2 (G), R13.2, R26.2
- new net: D10.1 (K), R24.1
- new net: R27.2, U9.10 (RX)
- new net: R25.2, U9.9 (TX)
- new net: D6.1 (K), R17.2
- new net: D9.1 (K), R23.2
- new net: U4.34 (OSC_OUT), Y1.1
- new net: U4.35 (OSC_IN), Y1.2
- new net GND: C1.2, C10.2, C11.2, C12.2, C13.2, C14.2, C15.2, C16.2, C17.2, C18.2, C19.2, C2.2, C20.2, C21.2, C22.2, C23.2, C24.2, C28.2, C30.2, C31.2, C34.2, C4.2, C5.2, C6.2, C7.2, C8.2, C9.2, D2.1 (A1), D5.1 (K), E1.1 (GND), E1.12 (GND), E1.24 (GND), E1.39 (GND), H1.1, H2.1, H3.1, H4.1, J1.3 (GND), J1.5 (GND), J1.6 (SWO/TDO), J1.8 (NC/TDI), J1.9 (GNDDetect), J11.5 (Pin_5), J15.3 (GND), J15.5 (GND), J15.6 (SWO/TDO), J15.8 (NC/TDI), J15.9 (GNDDetect), J3.A1 (GND), J3.A12 (GND), J3.B1 (GND), J3.B12 (GND), J4.1 (Pin_1), J5.1 (Pin_1), J5.3 (Pin_3), J6.1 (Pin_1), J6.3 (Pin_3), Q1.6, Q1.7, R1.2, R11.2, R16.2, R17.1, R18.1, R22.2, R23.1, R24.2, R4.1, R5.2, R6.2, R7.2, SW1.1, U1.2 (V_{SS}), U10.1 (CTG), U10.6 (QSTRT), U10.9 (EP), U11.3 (GND), U12.1 (GND), U3.13 (PS/SYNC), U3.15 (PGND), U3.2 (GND), U4.32 (VSSRF), U4.42 (VSSSMPS), U4.69 (VSS), U5.4 (GND), U6.2 (VSS), U7.2 (VSS), U8.5 (VCC), U9.12 (GND), U9.19 (GND), U9.3 (GND), U9.8 (GND)
Other:
- moved on the sheet: C20, D5, Q4, R13, R14, U9

Commit message: implement some feedback
Parts:
- removed R22: 1M, Resistor_SMD:R_0805_2012Metric_Pad1.20x1.40mm_HandSolder, symbol Device:R_US
Connections:
- net +VCC_OUT: now also U4.13 (VREF+)
- net GND: now also J3.S1 (SHIELD); no longer H1.1, H2.1, H3.1, H4.1, U3.13 (PS/SYNC)
- net at C6.1, U3.1 (VINA), U3.12 (EN): now also U3.13 (PS/SYNC)
